Commit message: 5/6

File: src/dynamic_reorient/urdf/ur5_with_gripper.urdf.xacro (robot description, xacro)
@@ -229,5 +229,5 @@
   <link name="camera_support">
     <visual>
-      <geometry><cylinder radius="0.008" length="0.20"/></geometry>
+      <geometry><cylinder radius="0.008" length="0.25"/></geometry>
       <material name="pole_grey"><color rgba="0.35 0.35 0.35 1.0"/></material>
     </visual>
@@ -243,5 +243,5 @@
     <parent link="world"/>
     <child link="camera_support"/>
-    <origin xyz="0.5 0 1.85" rpy="0 0 0"/>
+    <origin xyz="0.45 0 1.80" rpy="0 0 0"/>
   </joint>
   <link name="camera_link">
@@ -381,5 +381,5 @@
       <visualize>true</visualize>
       <camera>
-        <horizontal_fov>1.047</horizontal_fov>
+        <horizontal_fov>1.5708</horizontal_fov>
         <image>
           <width>640</width>
@@ -387,5 +387,5 @@
           <format>R8G8B8</format>
         </image>
-        <clip><near>0.1</near><far>3.0</far></clip>
+        <clip><near>0.1</near><far>5.0</far></clip>
       </camera>
       <plugin name="camera_plugin" filename="libgazebo_ros_camera.so">
@@ -393,5 +393,5 @@
         <frame_name>camera_optical_frame</frame_name>
         <min_depth>0.1</min_depth>
-        <max_depth>3.0</max_depth>
+        <max_depth>5.0</max_depth>
       </plugin>
     </sensor>
